Commit message: avance en diseño

File: mi_robot_description/urdf/mi_robot.urdf.xacro (robot description, xacro)
@@ -3,26 +3,41 @@
   <!-- Reusable Properties -->
   <!-- Chassis-->
-  <xacro:property name="chassis_length" value="0.4"/>
-  <xacro:property name="chassis_width" value="0.3"/>
-  <xacro:property name="chassis_height" value="0.1"/>
+  <xacro:property name="chassis_xlength" value="0.265"/>
+  <xacro:property name="chassis_ylength" value="0.094"/>
+  <xacro:property name="chassis_zlength" value="0.073"/>
+  <xacro:property name="chassis_mass" value="0.670"/>
+  <xacro:property name="chassis_zOfffset" value="0.015"/>
   <!-- Wheels-->
   <xacro:property name="wheel_radius" value="3.25"/>
   <xacro:property name="wheel_width" value="2.8"/>
+  <xacro:property name="wheel_xoffset" value="0.055"/>
+  <xacro:property name="wheel_mass" value="0.032"/>
+  <!-- Constants-->
+  <xacro:property name="pi" value="3.1415926535"/>
   <!-- Chasis -->
   <link name="base_link">
     <visual>
       <geometry>
-        <box size="${chassis_length} ${chassis_width} ${chassis_height}"/>
+        <box size="${chassis_xlength} ${chassis_ylength} ${chassis_zlength}"/>
       </geometry>
+      <origin xyz="0 0 ${chassis_zOfffset}" rpy="0 0 0"/>
       <material name="gray"><color rgba="0.5 0.5 0.5 1"/></material>
     </visual>
     <collision>
       <geometry>
-        <box size="${chassis_length} ${chassis_width} ${chassis_height}"/>
+        <box size="${chassis_xlength} ${chassis_ylength} ${chassis_zlength}"/>
       </geometry>
+      <origin xyz="0 0 ${chassis_zOfffset}" rpy="0 0 0"/>
     </collision>
     <inertial>
-      <mass value="5.0"/>
-      <inertia ixx="0.1" ixy="0" ixz="0" iyy="0.1" iyz="0" izz="0.1"/>
+    <origin xyz="0 0 ${chassis_zOfffset}" rpy="0 0 0"/>
+      <mass value="${chassis_mass}"/>
+      <inertia
+      ixx="$1/12*(chassis_ylength^2 + chassis_zlength^2)*chassis_mass"
+      ixy="0"
+      ixz="0"
+      iyy="$1/12*(chassis_xlength^2 + chassis_zlength^2)*chassis_mass"
+      iyz="0"
+      izz="$1/12*(chassis_xlength^2 + chassis_ylength^2)*chassis_mass"/>
     </inertial>
   </link>

Commit message: actualizacion variables ruedas

File: mi_robot_description/urdf/mi_robot.urdf.xacro (robot description, xacro)
@@ -9,7 +9,8 @@
   <xacro:property name="chassis_zOfffset" value="0.015"/>
   <!-- Wheels-->
-  <xacro:property name="wheel_radius" value="3.25"/>
-  <xacro:property name="wheel_width" value="2.8"/>
+  <xacro:property name="wheel_radius" value="0.0325"/>
+  <xacro:property name="wheel_width" value="0.028"/>
   <xacro:property name="wheel_xoffset" value="0.055"/>
+  <xacro:property name="wheel_yoffset" value="0.047"/>
   <xacro:property name="wheel_mass" value="0.032"/>
   <!-- Constants-->

Commit message: macros para ruedas

File: mi_robot_description/urdf/mi_robot.urdf.xacro (robot description, xacro)
@@ -14,4 +14,8 @@
   <xacro:property name="wheel_yoffset" value="0.047"/>
   <xacro:property name="wheel_mass" value="0.032"/>
+  <xacro:property name="wheel_Izz" value="${0.5*wheel_mass*wheel_radius*wheel_radius}"/>
+  <xacro:property name="wheel_Ixx" value="${(1.0/12.0)*wheel_mass*(3.0*wheel_radius*wheel_radius + wheel_width*wheel_width)}"/>
+  <xacro:property name="wheel_Iyy" value="${wheel_Ixx}"/>
+  <xacro:property name="wheel_Ixz" value="0"/>
   <!-- Constants-->
   <xacro:property name="pi" value="3.1415926535"/>
@@ -43,5 +47,5 @@
     </inertial>
   </link>
-  <!-- Macro para una rueda -->
+  <!-- Macro for a wheel -->
   <xacro:macro name="wheel_macro" params="wheel_name x y">
     <link name="${wheel_name}_link">
@@ -57,4 +61,15 @@
         </geometry>
       </collision>
+      <inertial>
+        <origin xyz="0 0 0" rpy="0 0 0"/>
+        <mass value="${wheel_mass}"/>
+        <inertia
+        ixx="$1/12*(3*wheel_radius^2 + wheel_width^2)*wheel_mass"
+        ixy="0"
+        ixz="0"
+        iyy="$1/12*(3*wheel_radius^2 + wheel_width^2)*wheel_mass"
+        iyz="0"
+        izz="$1/2*wheel_radius^2*wheel_mass"/>
+      </inertial>
     </link>
     <joint name="${wheel_name}_joint" type="continuous">

Commit message: revisar el tema de la altura de las ruedas

File: mi_robot_description/urdf/mi_robot.urdf.xacro (robot description, xacro)
@@ -12,5 +12,5 @@
   <xacro:property name="wheel_width" value="0.028"/>
   <xacro:property name="wheel_xoffset" value="0.055"/>
-  <xacro:property name="wheel_yoffset" value="0.047"/>
+  <xacro:property name="wheel_yoffset" value="${chassis_ylength/2 + wheel_width/2}"/>
   <xacro:property name="wheel_mass" value="0.032"/>
   <xacro:property name="wheel_Izz" value="${0.5*wheel_mass*wheel_radius*wheel_radius}"/>
@@ -81,8 +81,8 @@
   </xacro:macro>
   <!-- Ruedas (invocar macro) -->
-  <xacro:wheel_macro wheel_name="wheel_fl" x="${chassis_length/2 - wheel_width/2}" y="${chassis_width/2 - wheel_radius}"/>
-  <xacro:wheel_macro wheel_name="wheel_fr" x="${chassis_length/2 - wheel_width/2}" y="-${chassis_width/2 - wheel_radius}"/>
-  <xacro:wheel_macro wheel_name="wheel_rl" x="-${chassis_length/2 - wheel_width/2}" y="${chassis_width/2 - wheel_radius}"/>
-  <xacro:wheel_macro wheel_name="wheel_rr" x="-${chassis_length/2 - wheel_width/2}" y="-${chassis_width/2 - wheel_radius}"/>
+  <xacro:wheel_macro wheel_name="wheel_fl" x="${wheel_xoffset}" y="${wheel_yoffset}"/>
+  <xacro:wheel_macro wheel_name="wheel_fr" x="${wheel_xoffset}" y="${-wheel_yoffset}"/>
+  <xacro:wheel_macro wheel_name="wheel_rl" x="${-wheel_xoffset}" y="${wheel_yoffset}"/>
+  <xacro:wheel_macro wheel_name="wheel_rr" x="${-wheel_xoffset}" y="${-wheel_yoffset}"/>
   <!-- Sensor delantero -->
   <link name="sensor_front_link">

Commit message: mas cerca de que corra en rviz

File: mi_robot_description/urdf/mi_robot.urdf.xacro (robot description, xacro)
@@ -8,4 +8,10 @@
   <xacro:property name="chassis_mass" value="0.670"/>
   <xacro:property name="chassis_zOfffset" value="0.015"/>
+  <!-- Backwards-compatible aliases for older property names -->
+  <xacro:property name="chassis_length" value="${chassis_xlength}"/>
+  <xacro:property name="chassis_width" value="${chassis_ylength}"/>
+  <xacro:property name="chassis_height" value="${chassis_zlength}"/>
+  <!-- keep both spellings of zOffset (original had a typo) -->
+  <xacro:property name="chassis_zOffset" value="${chassis_zOfffset}"/>
   <!-- Wheels-->
   <xacro:property name="wheel_radius" value="0.0325"/>
@@ -18,6 +24,5 @@
   <xacro:property name="wheel_Iyy" value="${wheel_Ixx}"/>
   <xacro:property name="wheel_Ixz" value="0"/>
-  <!-- Constants-->
-  <xacro:property name="pi" value="3.1415926535"/>
+  <!-- Constants (avoid redefining common symbols) -->
   <!-- Chasis -->
   <link name="base_link">
@@ -36,15 +41,24 @@
     </collision>
     <inertial>
-    <origin xyz="0 0 ${chassis_zOfffset}" rpy="0 0 0"/>
+      <origin xyz="0 0 ${chassis_zOffset}" rpy="0 0 0"/>
       <mass value="${chassis_mass}"/>
       <inertia
-      ixx="$1/12*(chassis_ylength^2 + chassis_zlength^2)*chassis_mass"
-      ixy="0"
-      ixz="0"
-      iyy="$1/12*(chassis_xlength^2 + chassis_zlength^2)*chassis_mass"
-      iyz="0"
-      izz="$1/12*(chassis_xlength^2 + chassis_ylength^2)*chassis_mass"/>
+        ixx="${chassis_mass*(chassis_ylength*chassis_ylength + chassis_zlength*chassis_zlength)/12.0}"
+        ixy="0"
+        ixz="0"
+        iyy="${chassis_mass*(chassis_xlength*chassis_xlength + chassis_zlength*chassis_zlength)/12.0}"
+        iyz="0"
+        izz="${chassis_mass*(chassis_xlength*chassis_xlength + chassis_ylength*chassis_ylength)/12.0}"/>
     </inertial>
   </link>
+  <!-- Dummy root link to avoid KDL warning about inertia on root link -->
+  <link name="robot_root">
+    <!-- intentionally no inertial element here; KDL does not support inertia on the root link -->
+  </link>
+  <joint name="robot_root_joint" type="fixed">
+    <parent link="robot_root"/>
+    <child link="base_link"/>
+    <origin xyz="0 0 0" rpy="0 0 0"/>
+  </joint>
   <!-- Macro for a wheel -->
   <xacro:macro name="wheel_macro" params="wheel_name x y">
@@ -65,10 +79,10 @@
         <mass value="${wheel_mass}"/>
         <inertia
-        ixx="$1/12*(3*wheel_radius^2 + wheel_width^2)*wheel_mass"
-        ixy="0"
-        ixz="0"
-        iyy="$1/12*(3*wheel_radius^2 + wheel_width^2)*wheel_mass"
-        iyz="0"
-        izz="$1/2*wheel_radius^2*wheel_mass"/>
+          ixx="${wheel_mass*(3.0*wheel_radius*wheel_radius + wheel_width*wheel_width)/12.0}"
+          ixy="0"
+          ixz="0"
+          iyy="${wheel_mass*(3.0*wheel_radius*wheel_radius + wheel_width*wheel_width)/12.0}"
+          iyz="0"
+          izz="${0.5*wheel_mass*wheel_radius*wheel_radius}"/>
       </inertial>
     </link>
