Commit message: Add LiDAR support and update RViz configuration

File: mi_robot_description/urdf/mi_robot.urdf (robot description, URDF)
Before this commit: robot mi_robot, 8 links, 7 joints
Links:
- added link lidar_link, mass 0.05; collision cylinder length=0.04 radius=0.035; visual cylinder length=0.04 radius=0.035
Joints:
- added joint lidar_joint: type fixed, parent base_link, child lidar_link, origin xyz=0 0 0.056499999999999995 rpy=0 0 0

File: mi_robot_description/xacro/mi_robot.urdf.xacro (robot description, xacro)
@@ -24,4 +24,11 @@
   <xacro:property name="wheel_Iyy" value="${wheel_Ixx}"/>
   <xacro:property name="wheel_Ixz" value="0"/>
+<!-- LiDAR-->
+  <xacro:property name="lidar_length" value="0.04"/>
+  <xacro:property name="lidar_radius" value="0.035"/>
+  <xacro:property name="lidar_mass" value="0.05"/>
+  <xacro:property name="lidar_Izz" value="${0.5*lidar_mass*lidar_radius*lidar_radius}"/>
+  <xacro:property name="lidar_Ixx" value="${(1.0/12.0)*lidar_mass*(3.0*lidar_radius*lidar_radius + lidar_length*lidar_length)}"/>
+  <xacro:property name="lidar_Iyy" value="${lidar_Ixx}"/>
   <!-- Constants (avoid redefining common symbols) -->
   <xacro:property name="pi" value="3.14159265358979323846"/>
@@ -103,4 +110,34 @@
   <xacro:wheel_macro wheel_name="wheel_rl" x="${-wheel_xoffset}" y="${wheel_yoffset}"/>
   <xacro:wheel_macro wheel_name="wheel_rr" x="${-wheel_xoffset}" y="${-wheel_yoffset}"/>
+  <!-- LiDAR -->
+  <link name="lidar_link">
+    <visual>
+      <geometry>
+        <cylinder radius="${lidar_radius}" length="${lidar_length}"/>
+      </geometry>
+      <material name="green"><color rgba="0 1 0 1"/></material>
+     </visual>
+    <collision>
+      <geometry>
+        <cylinder radius="${lidar_radius}" length="${lidar_length}"/>
+      </geometry>
+    </collision>
+    <inertial>
+      <origin xyz="0 0 0" rpy="0 0 0"/>
+      <mass value="${lidar_mass}"/>
+      <inertia
+        ixx="${lidar_Ixx}"
+        ixy="0"
+        ixz="0"
+        iyy="${lidar_Iyy}"
+        iyz="0"
+        izz="${lidar_Izz}"/>
+    </inertial>
+  </link>
+  <joint name="lidar_joint" type="fixed">
+    <parent link="base_link"/>
+    <child link="lidar_link"/>
+    <origin xyz="0 0 ${chassis_height/2.0 + lidar_length/2.0}" rpy="0 0 0"/>
+  </joint>
   <!-- Sensor delantero -->
   <link name="sensor_front_link">

Commit message: Adjust wheel joint origins for improved alignment

File: mi_robot_description/urdf/mi_robot.urdf (robot description, URDF)
Before this commit: robot mi_robot, 9 links, 8 joints
Joints:
- joint wheel_fl_joint: origin xyz=0.055 0.061 -0.0365 rpy=0 0 0 -> xyz=0.055 0.061 -0.009125 rpy=0 0 0
- joint wheel_fr_joint: origin xyz=0.055 -0.061 -0.0365 rpy=0 0 0 -> xyz=0.055 -0.061 -0.009125 rpy=0 0 0
- joint wheel_rl_joint: origin xyz=-0.055 0.061 -0.0365 rpy=0 0 0 -> xyz=-0.055 0.061 -0.009125 rpy=0 0 0
- joint wheel_rr_joint: origin xyz=-0.055 -0.061 -0.0365 rpy=0 0 0 -> xyz=-0.055 -0.061 -0.009125 rpy=0 0 0

File: mi_robot_description/xacro/mi_robot.urdf.xacro (robot description, xacro)
@@ -100,5 +100,5 @@
       <parent link="base_link"/>
       <child link="${wheel_name}_link"/>
-      <origin xyz="${x} ${y} ${-chassis_height/2}" rpy="0 0 0"/>
+      <origin xyz="${x} ${y} ${-chassis_height/8}" rpy="0 0 0"/>
       <axis xyz="0 1 0"/>
       <limit effort="1.0" velocity="30"/>
