Commit message: basic model is visible on rviz2

File: mi_robot_description/xacro/mi_robot.urdf.xacro (robot description, xacro)
@@ -7,5 +7,5 @@
   <xacro:property name="chassis_zlength" value="0.073"/>
   <xacro:property name="chassis_mass" value="0.670"/>
-  <xacro:property name="chassis_zOfffset" value="0.015"/>
+  <xacro:property name="chassis_zOffset" value="0.015"/>
   <!-- Backwards-compatible aliases for older property names -->
   <xacro:property name="chassis_length" value="${chassis_xlength}"/>
@@ -13,5 +13,5 @@
   <xacro:property name="chassis_height" value="${chassis_zlength}"/>
   <!-- keep both spellings of zOffset (original had a typo) -->
-  <xacro:property name="chassis_zOffset" value="${chassis_zOfffset}"/>
+  <xacro:property name="chassis_zOfffset" value="${chassis_zOffset}"/>
   <!-- Wheels-->
   <xacro:property name="wheel_radius" value="0.0325"/>
@@ -25,4 +25,5 @@
   <xacro:property name="wheel_Ixz" value="0"/>
   <!-- Constants (avoid redefining common symbols) -->
+  <xacro:property name="pi" value="3.14159265358979323846"/>
   <!-- Chasis -->
   <link name="base_link">
@@ -31,5 +32,5 @@
         <box size="${chassis_xlength} ${chassis_ylength} ${chassis_zlength}"/>
       </geometry>
-      <origin xyz="0 0 ${chassis_zOfffset}" rpy="0 0 0"/>
+      <origin xyz="0 0 ${chassis_zOffset}" rpy="0 0 0"/>
       <material name="gray"><color rgba="0.5 0.5 0.5 1"/></material>
     </visual>
@@ -38,5 +39,5 @@
         <box size="${chassis_xlength} ${chassis_ylength} ${chassis_zlength}"/>
       </geometry>
-      <origin xyz="0 0 ${chassis_zOfffset}" rpy="0 0 0"/>
+      <origin xyz="0 0 ${chassis_zOffset}" rpy="0 0 0"/>
     </collision>
     <inertial>
@@ -65,4 +66,5 @@
     <link name="${wheel_name}_link">
       <visual>
+        <origin xyz="0 0 0" rpy="${pi/2} 0 0"/>
         <geometry>
           <cylinder radius="${wheel_radius}" length="${wheel_width}"/>
@@ -71,4 +73,5 @@
       </visual>
       <collision>
+        <origin xyz="0 0 0" rpy="${pi/2} 0 0"/>
         <geometry>
           <cylinder radius="${wheel_radius}" length="${wheel_width}"/>
@@ -76,5 +79,5 @@
       </collision>
       <inertial>
-        <origin xyz="0 0 0" rpy="0 0 0"/>
+        <origin xyz="0 0 0" rpy="${pi/2} 0 0"/>
         <mass value="${wheel_mass}"/>
         <inertia
@@ -92,4 +95,5 @@
       <origin xyz="${x} ${y} ${-chassis_height/2}" rpy="0 0 0"/>
       <axis xyz="0 1 0"/>
+      <limit effort="1.0" velocity="30"/>
     </joint>
   </xacro:macro>
@@ -111,5 +115,5 @@
     <parent link="base_link"/>
     <child link="sensor_front_link"/>
-    <origin xyz="${chassis_length/2 + 0.02} 0 ${chassis_height/2}" rpy="0 0 0"/>
+    <origin xyz="${(chassis_length/2.0) + 0.02} 0 ${chassis_height/2.0}" rpy="0 0 0"/>
   </joint>
   <!-- Sensor trasero -->
@@ -125,5 +129,5 @@
     <parent link="base_link"/>
     <child link="sensor_back_link"/>
-    <origin xyz="-${chassis_length/2 + 0.02} 0 ${chassis_height/2}" rpy="0 0 0"/>
+    <origin xyz="${-(chassis_length/2.0 + 0.02)} 0 ${chassis_height/2.0}" rpy="0 0 0"/>
   </joint>
 </robot>

Commit message: gazebo config files

File: mi_robot_description/xacro/mi_robot.urdf.xacro (robot description, xacro)
@@ -32,5 +32,5 @@
   <xacro:property name="lidar_Iyy" value="${lidar_Ixx}"/>
   <!-- Constants (avoid redefining common symbols) -->
-  <xacro:property name="pi" value="3.14159265358979323846"/>
+  <!-- xacro:property name="pi" value="3.141592653589793"/-->
   <!-- Chasis -->
   <link name="base_link">
@@ -168,37 +168,5 @@
     <origin xyz="${-(chassis_length/2.0 + 0.02)} 0 ${chassis_height/2.0}" rpy="0 0 0"/>
   </joint>
-<!--gazebo-->
-<plugin filename="gz-sim-sensors-system" name="gz::sim::systems::Sensors">
-  <render_engine>ogre2</render_engine>
-</plugin>
-<gazebo reference= "lidar_link">
-  <sensor name="gpu_lidar" type = "gpu_lidar"> <!--if there's no gpu just use ray-->
-    	<pose> 0 0 0 0 0 0 </pose>
-    	<visualize> true </visualize>
-    	<update_rate> 10 </update_rate>
-		<topic> scan </topic>
-    	<lidar>
-			<scan>
-				<horizontal>
-					<samples> 360 </samples>
-					<resolution> 1 </resolution>
-					<min_angle> ${-pi} </min_angle>
-					<max_angle> ${pi} </max_angle>
-				</horizontal>
-			</scan>
-			<range>
-				<min> 0.3 </min>
-				<max> 12 </max>
-				<resolution> 0.01 </resolution>
-			</range>
-		    <noise>
-				<type> gaussian </type>
-				<mean> 0.0 </mean>
-				<stddev> 0.01 </stddev>
-			</noise>
-		</lidar>
-		<always_on> true </always_on>
-		<visualize> true </visualize>
-    </sensor>
-</gazebo>
+  <!-- Incluir las definiciones de Gazebo -->
+  <xacro:include filename="$(find mi_robot_description)/xacro/mi_robot.gazebo.xacro" />
 </robot>
