Commit message: imu configuration yet not working properly

File: mi_robot_description/xacro/mi_robot.gazebo.xacro (robot description, xacro)
@@ -31,4 +31,67 @@
         </sensor>
     </gazebo>
+    <!-- IMU -->
+    <gazebo reference="imu_link">
+    <sensor name="imu_sensor" type="imu">
+        <always_on>1</always_on>
+        <update_rate>50</update_rate>
+        <topic>/imu/data</topic>
+        <imu>
+          <!-- El bloque <imu> solo contiene el modelo de ruido -->
+          <angular_velocity>
+            <x>
+              <noise type="gaussian">
+                <mean>0.0</mean>
+                <stddev>2e-4</stddev>
+                <bias_mean>0.0000075</bias_mean>
+                <bias_stddev>0.0000008</bias_stddev>
+              </noise>
+            </x>
+            <y>
+              <noise type="gaussian">
+                <mean>0.0</mean>
+                <stddev>2e-4</stddev>
+                <bias_mean>0.0000075</bias_mean>
+                <bias_stddev>0.0000008</bias_stddev>
+              </noise>
+            </y>
+            <z>
+              <noise type="gaussian">
+                <mean>0.0</mean>
+                <stddev>2e-4</stddev>
+                <bias_mean>0.0000075</bias_mean>
+                <bias_stddev>0.0000008</bias_stddev>
+              </noise>
+            </z>
+          </angular_velocity>
+          <linear_acceleration>
+            <x>
+              <noise type="gaussian">
+                <mean>0.0</mean>
+                <stddev>1.7e-2</stddev>
+                <bias_mean>0.1</bias_mean>
+                <bias_stddev>0.001</bias_stddev>
+              </noise>
+            </x>
+            <y>
+              <noise type="gaussian">
+                <mean>0.0</mean>
+                <stddev>1.7e-2</stddev>
+                <bias_mean>0.1</bias_mean>
+                <bias_stddev>0.001</bias_stddev>
+              </noise>
+            </y>
+            <z>
+              <noise type="gaussian">
+                <mean>0.0</mean>
+                <stddev>1.7e-2</stddev>
+                <bias_mean>0.1</bias_mean>
+                <bias_stddev>0.001</bias_stddev>
+              </noise>
+            </z>
+          </linear_acceleration>
+        </imu>
+    </sensor>
+</gazebo>
     <!-- Plugin para el controlador de tracción diferencial (DiffDrive) -->
     <gazebo>

File: mi_robot_description/xacro/mi_robot.urdf.xacro (robot description, xacro)
@@ -31,4 +31,9 @@
   <xacro:property name="lidar_Ixx" value="${(1.0/12.0)*lidar_mass*(3.0*lidar_radius*lidar_radius + lidar_length*lidar_length)}"/>
   <xacro:property name="lidar_Iyy" value="${lidar_Ixx}"/>
+  <!--IMU-->
+  <xacro:property name="imu_mass" value="0.02"/>
+  <xacro:property name="imu_xlength" value="0.02"/>
+  <xacro:property name="imu_ylength" value="0.02"/>
+  <xacro:property name="imu_zlength" value="0.02"/>
   <!-- Constants (avoid redefining common symbols) -->
   <!-- Chasis -->
@@ -115,5 +120,5 @@
         <cylinder radius="${lidar_radius}" length="${lidar_length}"/>
       </geometry>
-      <material name="green"><color rgba="0 1 0 1"/></material>
+      <material name="black"><color rgba="0 0 0 1"/></material>
      </visual>
     <collision>
@@ -139,4 +144,29 @@
     <origin xyz="0 0 ${chassis_height/2.0 + lidar_length/2.0}" rpy="0 0 0"/>
   </joint>
+  <!-- imu -->
+  <link name="imu_link">
+    <visual>
+      <geometry>
+        <box size="${imu_xlength} ${imu_ylength} ${imu_zlength}"/>
+      </geometry>
+      <material name="yellow"><color rgba="1 1 0 1"/></material>
+    </visual>
+    <inertial>
+      <origin xyz="0 0 0" rpy="0 0 0"/>
+      <mass value="${imu_mass}"/>
+      <inertia
+        ixx="${imu_mass*(imu_ylength*imu_ylength + imu_zlength*imu_zlength)/12.0}"
+        ixy="0"
+        ixz="0"
+        iyy="${imu_mass*(imu_xlength*imu_xlength + imu_zlength*imu_zlength)/12.0}"
+        iyz="0"
+        izz="${imu_mass*(imu_xlength*imu_xlength + imu_ylength*imu_ylength)/12.0}"/>
+    </inertial>
+  </link>
+  <joint name="imu_joint" type="fixed">
+    <parent link="base_link"/>
+    <child link="imu_link"/>
+    <origin xyz="0 0 ${chassis_zlength/2.0}" rpy="0 0 0"/>
+  </joint>
   <!-- Sensor delantero -->
   <link name="sensor_front_link">
